File: Power_supply.kicad_pcb (KiCad board)
At the start: 2 copper layers, 30.1 x 52.1 mm, 15 parts, among them J1 Barrel_Jack_Switch, J2 Conn_02x02_Odd_Even, J3 Conn_02x02_Odd_Even, SW1 SW_DPDT_x2, U1 LM7805_TO220

Commit message: add gerber files
Other:
- board text added: "5v"
- board text added: "Breadboard Power supply v1.0"
- board text added: "GND"
Changed lines of the file:
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@@
   (general
     (thickness 1.6)
-    (drawings 8)
+    (drawings 13)
     (tracks 51)
     (zones 0)
@@
     (descr "CP, Radial series, Radial, pin pitch=5.00mm, , diameter=10mm, Electrolytic Capacitor")
     (tags "CP Radial series Radial pin pitch 5.00mm  diameter 10mm Electrolytic Capacitor")
-    (fp_text reference C1 (at 2.5 -6.25) (layer F.SilkS)
+    (fp_text reference C1 (at -1.72 -4.69) (layer F.SilkS)
       (effects (font (size 1 1) (thickness 0.15)))
     )
@@
     (descr "CP, Radial series, Radial, pin pitch=2.50mm, , diameter=6.3mm, Electrolytic Capacitor")
     (tags "CP Radial series Radial pin pitch 2.50mm  diameter 6.3mm Electrolytic Capacitor")
-    (fp_text reference C2 (at 1.25 -4.4) (layer F.SilkS)
+    (fp_text reference C2 (at -3.14 -2.68) (layer F.SilkS)
       (effects (font (size 1 1) (thickness 0.15)))
     )
@@
       (effects (font (size 1 1) (thickness 0.15)))
     )
-    (fp_text user K (at 0 -2.1) (layer F.Fab)
-      (effects (font (size 1 1) (thickness 0.15)))
-    )
-    (fp_text user K (at 0 -2.1) (layer F.SilkS)
-      (effects (font (size 1 1) (thickness 0.15)))
-    )
     (pad 1 thru_hole rect (at 0 0) (size 2.2 2.2) (drill 1.1) (layers *.Cu *.Mask)
       (net 1 /Vin))
@@
     (fp_line (start 11.51 1.6) (end 11.51 -1.6) (layer F.CrtYd) (width 0.05))
     (fp_line (start 11.51 -1.6) (end -1.35 -1.6) (layer F.CrtYd) (width 0.05))
-    (fp_text user K (at 0 -2.1) (layer F.SilkS)
-      (effects (font (size 1 1) (thickness 0.15)))
-    )
-    (fp_text user K (at 0 -2.1) (layer F.Fab)
-      (effects (font (size 1 1) (thickness 0.15)))
-    )
     (fp_text user %R (at 5.47 0) (layer F.Fab)
       (effects (font (size 1 1) (thickness 0.15)))
@@
     (fp_line (start 11.51 1.6) (end 11.51 -1.6) (layer F.CrtYd) (width 0.05))
     (fp_line (start 11.51 -1.6) (end -1.35 -1.6) (layer F.CrtYd) (width 0.05))
-    (fp_text user K (at 0 -2.1) (layer F.SilkS)
-      (effects (font (size 1 1) (thickness 0.15)))
-    )
-    (fp_text user K (at 0 -2.1) (layer F.Fab)
-      (effects (font (size 1 1) (thickness 0.15)))
-    )
     (fp_text user %R (at 5.47 0) (layer F.Fab)
       (effects (font (size 1 1) (thickness 0.15)))
@@
       (effects (font (size 1 1) (thickness 0.15)))
     )
+    (fp_text user %R (at 5.47 0) (layer F.Fab)
+      (effects (font (size 1 1) (thickness 0.15)))
+    )
+    (fp_line (start 2.48 -1.35) (end 2.48 1.35) (layer F.Fab) (width 0.1))
+    (fp_line (start 2.48 1.35) (end 7.68 1.35) (layer F.Fab) (width 0.1))
+    (fp_line (start 7.68 1.35) (end 7.68 -1.35) (layer F.Fab) (width 0.1))
+    (fp_line (start 7.68 -1.35) (end 2.48 -1.35) (layer F.Fab) (width 0.1))
+    (fp_line (start 0 0) (end 2.48 0) (layer F.Fab) (width 0.1))
+    (fp_line (start 10.16 0) (end 7.68 0) (layer F.Fab) (width 0.1))
+    (fp_line (start 3.26 -1.35) (end 3.26 1.35) (layer F.Fab) (width 0.1))
+    (fp_line (start 3.36 -1.35) (end 3.36 1.35) (layer F.Fab) (width 0.1))
+    (fp_line (start 3.16 -1.35) (end 3.16 1.35) (layer F.Fab) (width 0.1))
+    (fp_line (start 2.36 -1.47) (end 2.36 1.47) (layer F.SilkS) (width 0.12))
+    (fp_line (start 2.36 1.47) (end 7.8 1.47) (layer F.SilkS) (width 0.12))
+    (fp_line (start 7.8 1.47) (end 7.8 -1.47) (layer F.SilkS) (width 0.12))
+    (fp_line (start 7.8 -1.47) (end 2.36 -1.47) (layer F.SilkS) (width 0.12))
+    (fp_line (start 1.34 0) (end 2.36 0) (layer F.SilkS) (width 0.12))
+    (fp_line (start 8.82 0) (end 7.8 0) (layer F.SilkS) (width 0.12))
+    (fp_line (start 3.26 -1.47) (end 3.26 1.47) (layer F.SilkS) (width 0.12))
+    (fp_line (start 3.38 -1.47) (end 3.38 1.47) (layer F.SilkS) (width 0.12))
+    (fp_line (start 3.14 -1.47) (end 3.14 1.47) (layer F.SilkS) (width 0.12))
+    (fp_line (start -1.35 -1.6) (end -1.35 1.6) (layer F.CrtYd) (width 0.05))
+    (fp_line (start -1.35 1.6) (end 11.51 1.6) (layer F.CrtYd) (width 0.05))
+    (fp_line (start 11.51 1.6) (end 11.51 -1.6) (layer F.CrtYd) (width 0.05))
     (fp_line (start 11.51 -1.6) (end -1.35 -1.6) (layer F.CrtYd) (width 0.05))
-    (fp_line (start 11.51 1.6) (end 11.51 -1.6) (layer F.CrtYd) (width 0.05))
-    (fp_line (start -1.35 1.6) (end 11.51 1.6) (layer F.CrtYd) (width 0.05))
-    (fp_line (start -1.35 -1.6) (end -1.35 1.6) (layer F.CrtYd) (width 0.05))
-    (fp_line (start 3.14 -1.47) (end 3.14 1.47) (layer F.SilkS) (width 0.12))
-    (fp_line (start 3.38 -1.47) (end 3.38 1.47) (layer F.SilkS) (width 0.12))
-    (fp_line (start 3.26 -1.47) (end 3.26 1.47) (layer F.SilkS) (width 0.12))
-    (fp_line (start 8.82 0) (end 7.8 0) (layer F.SilkS) (width 0.12))
-    (fp_line (start 1.34 0) (end 2.36 0) (layer F.SilkS) (width 0.12))
-    (fp_line (start 7.8 -1.47) (end 2.36 -1.47) (layer F.SilkS) (width 0.12))
-    (fp_line (start 7.8 1.47) (end 7.8 -1.47) (layer F.SilkS) (width 0.12))
-    (fp_line (start 2.36 1.47) (end 7.8 1.47) (layer F.SilkS) (width 0.12))
-    (fp_line (start 2.36 -1.47) (end 2.36 1.47) (layer F.SilkS) (width 0.12))
-    (fp_line (start 3.16 -1.35) (end 3.16 1.35) (layer F.Fab) (width 0.1))
-    (fp_line (start 3.36 -1.35) (end 3.36 1.35) (layer F.Fab) (width 0.1))
-    (fp_line (start 3.26 -1.35) (end 3.26 1.35) (layer F.Fab) (width 0.1))
-    (fp_line (start 10.16 0) (end 7.68 0) (layer F.Fab) (width 0.1))
-    (fp_line (start 0 0) (end 2.48 0) (layer F.Fab) (width 0.1))
-    (fp_line (start 7.68 -1.35) (end 2.48 -1.35) (layer F.Fab) (width 0.1))
-    (fp_line (start 7.68 1.35) (end 7.68 -1.35) (layer F.Fab) (width 0.1))
-    (fp_line (start 2.48 1.35) (end 7.68 1.35) (layer F.Fab) (width 0.1))
-    (fp_line (start 2.48 -1.35) (end 2.48 1.35) (layer F.Fab) (width 0.1))
-    (fp_text user %R (at 5.47 0) (layer F.Fab)
-      (effects (font (size 1 1) (thickness 0.15)))
-    )
-    (fp_text user K (at 0 -2.1) (layer F.Fab)
-      (effects (font (size 1 1) (thickness 0.15)))
-    )
-    (fp_text user K (at 0 -2.1) (layer F.SilkS)
-      (effects (font (size 1 1) (thickness 0.15)))
-    )
+    (pad 2 thru_hole oval (at 10.16 0) (size 2.2 2.2) (drill 1.1) (layers *.Cu *.Mask)
+      (net 2 /V-))
     (pad 1 thru_hole rect (at 0 0) (size 2.2 2.2) (drill 1.1) (layers *.Cu *.Mask)
       (net 5 "Net-(D3-Pad2)"))
-    (pad 2 thru_hole oval (at 10.16 0) (size 2.2 2.2) (drill 1.1) (layers *.Cu *.Mask)
-      (net 2 /V-))
     (model ${KISYS3DMOD}/Diode_THT.3dshapes/D_DO-41_SOD81_P10.16mm_Horizontal.wrl
       (at (xyz 0 0 0))
@@
     (descr "Through hole straight pin header, 2x02, 2.54mm pitch, double rows")
     (tags "Through hole pin header THT 2x02 2.54mm double row")
-    (fp_text reference J2 (at 1.27 -2.33) (layer F.SilkS)
+    (fp_text reference J2 (at -2.55 1.38 90) (layer F.SilkS)
       (effects (font (size 1 1) (thickness 0.15)))
     )
@@
     (descr "Through hole straight pin header, 2x02, 2.54mm pitch, double rows")
     (tags "Through hole pin header THT 2x02 2.54mm double row")
-    (fp_text reference J3 (at 1.27 -2.33) (layer F.SilkS)
+    (fp_text reference J3 (at -2.44 1.41 90) (layer F.SilkS)
       (effects (font (size 1 1) (thickness 0.15)))
     )
@@
     (descr "Resistor, Axial_DIN0207 series, Axial, Horizontal, pin pitch=7.62mm, 0.25W = 1/4W, length*diameter=6.3*2.5mm^2, http://cdn-reichelt.de/documents/datenblatt/B400/1_4W%23YAG.pdf")
     (tags "Resistor Axial_DIN0207 series Axial Horizontal pin pitch 7.62mm 0.25W = 1/4W length 6.3mm diameter 2.5mm")
-    (fp_text reference R1 (at 3.81 -2.37 90) (layer F.SilkS)
+    (fp_text reference R1 (at 6.57 -2.12 90) (layer F.SilkS)
       (effects (font (size 1 1) (thickness 0.15)))
     )
@@
     (descr "Resistor, Axial_DIN0207 series, Axial, Horizontal, pin pitch=7.62mm, 0.25W = 1/4W, length*diameter=6.3*2.5mm^2, http://cdn-reichelt.de/documents/datenblatt/B400/1_4W%23YAG.pdf")
     (tags "Resistor Axial_DIN0207 series Axial Horizontal pin pitch 7.62mm 0.25W = 1/4W length 6.3mm diameter 2.5mm")
-    (fp_text reference R2 (at 3.81 -2.37 90) (layer F.SilkS)
+    (fp_text reference R2 (at 1.12 -2.21 90) (layer F.SilkS)
       (effects (font (size 1 1) (thickness 0.15)))
     )
@@
     )
   )
+  (gr_text 5v (at 140.61 83.06) (layer F.SilkS)
+    (effects (font (size 1 1.4) (thickness 0.15)))
+  )
+  (gr_text GND (at 140.31 86.96) (layer F.SilkS)
+    (effects (font (size 1 1) (thickness 0.15)))
+  )
+  (gr_text GND (at 140.52 131.97) (layer F.SilkS)
+    (effects (font (size 1 1) (thickness 0.15)))
+  )
+  (gr_text 5v (at 140.82 128.07) (layer F.SilkS)
+    (effects (font (size 1 1.4) (thickness 0.15)))
+  )
+  (gr_text "Breadboard\nPower supply\nv1.0\n" (at 121.55 127.06 90) (layer B.SilkS)
+    (effects (font (size 1 1) (thickness 0.25)) (justify mirror))
+  )
   (gr_line (start 141.986 88.265) (end 141.986 126.365) (layer Edge.Cuts) (width 0.05))
